File: Ekogolf-board.brd (EAGLE design)
At the start: 84.8 x 64.8 mm, 10 parts

Commit message: first routing
Parts:
- moved X2 50.8 mm to (11.4, 34.3)
- moved X7 21.6 mm to (61.0, 34.3)
- moved X6 20.4 mm to (34.3, 34.3)
Connections:
- removed net N$2: SV2.6
- net N$1: no longer X2.1
Routing:
- net N$1: track 0.00 -> 155.3 mm
- net N$3: track 0.00 -> 93.5 mm
Other:
- board size 84.8 x 64.8 mm -> 84.8 x 63.5 mm
Changed lines of the file:
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@@
 <board>
 <plain>
-<wire x1="-7.62" y1="1.27" x2="77.14" y2="1.27" width="0" layer="20"/>
-<wire x1="77.14" y1="1.27" x2="77.14" y2="66.03" width="0" layer="20"/>
+<wire x1="-7.62" y1="2.54" x2="77.14" y2="2.54" width="0" layer="20"/>
+<wire x1="77.14" y1="2.54" x2="77.14" y2="66.03" width="0" layer="20"/>
 <wire x1="77.14" y1="66.03" x2="-7.62" y2="66.03" width="0" layer="20"/>
-<wire x1="-7.62" y1="66.03" x2="-7.62" y2="1.27" width="0" layer="20"/>
+<wire x1="-7.62" y1="66.03" x2="-7.62" y2="2.54" width="0" layer="20"/>
 </plain>
 <attributes>
@@
 <attribute name="VALUE" x="7.62" y="44.49" size="1.27" layer="27" ratio="10" rot="R90"/>
 </element>
-<element name="X6" library="con-wago-500" library_urn="urn:adsk.eagle:library:195" package="W237-4" package3d_urn="urn:adsk.eagle:package:10695/1" value="" x="13.97" y="35.56" smashed="yes">
-<attribute name="MF" value="" x="13.97" y="35.56" size="1.778" layer="27" display="off"/>
-<attribute name="MPN" value="" x="13.97" y="35.56" size="1.778" layer="27" display="off"/>
-<attribute name="NAME" x="5.2254" y="28.1178" size="1.27" layer="25" ratio="10"/>
-<attribute name="OC_FARNELL" value="unknown" x="13.97" y="35.56" size="1.778" layer="27" display="off"/>
-<attribute name="OC_NEWARK" value="unknown" x="13.97" y="35.56" size="1.778" layer="27" display="off"/>
-<attribute name="VALUE" x="6.3176" y="30.5308" size="1.27" layer="27" ratio="10"/>
-</element>
-<element name="X7" library="con-wago-500" library_urn="urn:adsk.eagle:library:195" package="W237-4" package3d_urn="urn:adsk.eagle:package:10695/1" value="" x="39.37" y="35.56" smashed="yes">
-<attribute name="MF" value="" x="39.37" y="35.56" size="1.778" layer="27" display="off"/>
-<attribute name="MPN" value="" x="39.37" y="35.56" size="1.778" layer="27" display="off"/>
-<attribute name="NAME" x="30.6254" y="28.1178" size="1.27" layer="25" ratio="10"/>
-<attribute name="OC_FARNELL" value="unknown" x="39.37" y="35.56" size="1.778" layer="27" display="off"/>
-<attribute name="OC_NEWARK" value="unknown" x="39.37" y="35.56" size="1.778" layer="27" display="off"/>
-<attribute name="VALUE" x="31.7176" y="30.5308" size="1.27" layer="27" ratio="10"/>
-</element>
-<element name="X2" library="con-wago-500" library_urn="urn:adsk.eagle:library:195" package="W237-103" package3d_urn="urn:adsk.eagle:package:10691/1" value="" x="62.23" y="35.56" smashed="yes">
-<attribute name="MF" value="" x="62.23" y="35.56" size="1.778" layer="27" display="off"/>
-<attribute name="MPN" value="237-103" x="62.23" y="35.56" size="1.778" layer="27" display="off"/>
-<attribute name="NAME" x="56.5442" y="28.0978" size="1.27" layer="25" ratio="10"/>
-<attribute name="OC_FARNELL" value="unknown" x="62.23" y="35.56" size="1.778" layer="27" display="off"/>
-<attribute name="OC_NEWARK" value="18M7116" x="62.23" y="35.56" size="1.778" layer="27" display="off"/>
-<attribute name="VALUE" x="56.9252" y="30.6124" size="1.27" layer="27" ratio="10"/>
+<element name="X6" library="con-wago-500" library_urn="urn:adsk.eagle:library:195" package="W237-4" package3d_urn="urn:adsk.eagle:package:10695/1" value="" x="34.29" y="34.29" smashed="yes">
+<attribute name="MF" value="" x="34.29" y="34.29" size="1.778" layer="27" display="off"/>
+<attribute name="MPN" value="" x="34.29" y="34.29" size="1.778" layer="27" display="off"/>
+<attribute name="NAME" x="25.5454" y="26.8478" size="1.27" layer="25" ratio="10"/>
+<attribute name="OC_FARNELL" value="unknown" x="34.29" y="34.29" size="1.778" layer="27" display="off"/>
+<attribute name="OC_NEWARK" value="unknown" x="34.29" y="34.29" size="1.778" layer="27" display="off"/>
+<attribute name="VALUE" x="26.6376" y="29.2608" size="1.27" layer="27" ratio="10"/>
+</element>
+<element name="X7" library="con-wago-500" library_urn="urn:adsk.eagle:library:195" package="W237-4" package3d_urn="urn:adsk.eagle:package:10695/1" value="" x="60.96" y="34.29" smashed="yes">
+<attribute name="MF" value="" x="60.96" y="34.29" size="1.778" layer="27" display="off"/>
+<attribute name="MPN" value="" x="60.96" y="34.29" size="1.778" layer="27" display="off"/>
+<attribute name="NAME" x="52.2154" y="26.8478" size="1.27" layer="25" ratio="10"/>
+<attribute name="OC_FARNELL" value="unknown" x="60.96" y="34.29" size="1.778" layer="27" display="off"/>
+<attribute name="OC_NEWARK" value="unknown" x="60.96" y="34.29" size="1.778" layer="27" display="off"/>
+<attribute name="VALUE" x="53.3076" y="29.2608" size="1.27" layer="27" ratio="10"/>
+</element>
+<element name="X2" library="con-wago-500" library_urn="urn:adsk.eagle:library:195" package="W237-103" package3d_urn="urn:adsk.eagle:package:10691/1" value="" x="11.43" y="34.29" smashed="yes">
+<attribute name="MF" value="" x="11.43" y="34.29" size="1.778" layer="27" display="off"/>
+<attribute name="MPN" value="237-103" x="11.43" y="34.29" size="1.778" layer="27" display="off"/>
+<attribute name="NAME" x="5.7442" y="26.8278" size="1.27" layer="25" ratio="10"/>
+<attribute name="OC_FARNELL" value="unknown" x="11.43" y="34.29" size="1.778" layer="27" display="off"/>
+<attribute name="OC_NEWARK" value="18M7116" x="11.43" y="34.29" size="1.778" layer="27" display="off"/>
+<attribute name="VALUE" x="6.1252" y="29.3424" size="1.27" layer="27" ratio="10"/>
 </element>
 </elements>
@@
 <contactref element="X7" pad="1"/>
 <contactref element="SV1" pad="5"/>
-<contactref element="X2" pad="1"/>
-<wire x1="31.87" y1="34.29" x2="57.23" y2="34.27" width="0" layer="19" extent="1-1"/>
-<wire x1="6.47" y1="34.29" x2="31.87" y2="34.29" width="0" layer="19" extent="1-1"/>
-<wire x1="19.05" y1="10.16" x2="6.47" y2="34.29" width="0" layer="19" extent="1-1"/>
+<wire x1="53.46" y1="33.02" x2="53.46" y2="31.87" width="0.1524" layer="16"/>
+<wire x1="53.46" y1="31.87" x2="53.34" y2="31.75" width="0.1524" layer="16"/>
+<wire x1="53.34" y1="31.75" x2="54.61" y2="30.48" width="0.1524" layer="16"/>
+<wire x1="54.61" y1="30.48" x2="64.77" y2="30.48" width="0.1524" layer="16"/>
+<wire x1="64.77" y1="30.48" x2="66.04" y2="31.75" width="0.1524" layer="16"/>
+<wire x1="66.04" y1="35.56" x2="67.31" y2="36.83" width="0.1524" layer="16"/>
+<wire x1="67.31" y1="36.83" x2="71.12" y2="36.83" width="0.1524" layer="16"/>
+<wire x1="71.12" y1="36.83" x2="72.39" y2="35.56" width="0.1524" layer="16"/>
+<wire x1="53.34" y1="16.51" x2="52.07" y2="15.24" width="0.1524" layer="16"/>
+<wire x1="52.07" y1="15.24" x2="52.07" y2="7.62" width="0.1524" layer="16"/>
+<wire x1="52.07" y1="7.62" x2="49.53" y2="5.08" width="0.1524" layer="16"/>
+<wire x1="49.53" y1="5.08" x2="20.32" y2="5.08" width="0.1524" layer="16"/>
+<wire x1="20.32" y1="5.08" x2="19.05" y2="6.35" width="0.1524" layer="16"/>
+<wire x1="19.05" y1="6.35" x2="19.05" y2="10.16" width="0.1524" layer="16"/>
+<wire x1="66.04" y1="31.75" x2="66.04" y2="35.56" width="0.1524" layer="16"/>
+<wire x1="72.39" y1="35.56" x2="72.39" y2="19.05" width="0.1524" layer="16"/>
+<wire x1="72.39" y1="19.05" x2="69.85" y2="16.51" width="0.1524" layer="16"/>
+<wire x1="69.85" y1="16.51" x2="53.34" y2="16.51" width="0.1524" layer="16"/>
+<wire x1="26.79" y1="33.02" x2="26.67" y2="33.14" width="0.1524" layer="16"/>
+<wire x1="26.67" y1="33.14" x2="26.67" y2="34.29" width="0.1524" layer="16"/>
+<wire x1="26.67" y1="34.29" x2="24.13" y2="36.83" width="0.1524" layer="16"/>
+<wire x1="24.13" y1="36.83" x2="15.24" y2="36.83" width="0.1524" layer="16"/>
+<wire x1="15.24" y1="36.83" x2="13.97" y2="35.56" width="0.1524" layer="16"/>
+<wire x1="13.97" y1="19.05" x2="15.24" y2="17.78" width="0.1524" layer="16"/>
+<wire x1="15.24" y1="17.78" x2="17.78" y2="17.78" width="0.1524" layer="16"/>
+<wire x1="17.78" y1="17.78" x2="19.05" y2="16.51" width="0.1524" layer="16"/>
+<wire x1="13.97" y1="35.56" x2="13.97" y2="19.05" width="0.1524" layer="16"/>
+<wire x1="19.05" y1="16.51" x2="19.05" y2="10.16" width="0.1524" layer="16"/>
 </signal>
 <signal name="N$3">
@@
 <contactref element="SV1" pad="6"/>
 <contactref element="X2" pad="3"/>
-<wire x1="46.87" y1="34.29" x2="67.23" y2="34.27" width="0" layer="19" extent="1-1"/>
-<wire x1="21.47" y1="34.29" x2="46.87" y2="34.29" width="0" layer="19" extent="1-1"/>
-<wire x1="21.59" y1="10.16" x2="21.47" y2="34.29" width="0" layer="19" extent="1-1"/>
-</signal>
-<signal name="N$2">
-<contactref element="SV2" pad="6"/>
+<wire x1="41.79" y1="33.02" x2="41.79" y2="29.33" width="0.1524" layer="16"/>
+<wire x1="67.31" y1="27.94" x2="68.58" y2="29.21" width="0.1524" layer="16"/>
+<wire x1="68.58" y1="32.9" x2="68.46" y2="33.02" width="0.1524" layer="16"/>
+<wire x1="41.79" y1="29.33" x2="43.18" y2="27.94" width="0.1524" layer="16"/>
+<wire x1="43.18" y1="27.94" x2="67.31" y2="27.94" width="0.1524" layer="16"/>
+<wire x1="68.58" y1="29.21" x2="68.58" y2="32.9" width="0.1524" layer="16"/>
+<wire x1="21.59" y1="10.16" x2="21.59" y2="12.7" width="0.1524" layer="16"/>
+<wire x1="21.59" y1="12.7" x2="24.13" y2="15.24" width="0.1524" layer="16"/>
+<wire x1="24.13" y1="15.24" x2="39.37" y2="15.24" width="0.1524" layer="16"/>
+<wire x1="43.18" y1="19.05" x2="43.18" y2="27.94" width="0.1524" layer="16"/>
+<wire x1="39.37" y1="15.24" x2="43.18" y2="19.05" width="0.1524" layer="16"/>
+<wire x1="16.43" y1="33" x2="16.51" y2="32.92" width="0.1524" layer="16"/>
+<wire x1="20.32" y1="24.13" x2="22.86" y2="24.13" width="0.1524" layer="16"/>
+<wire x1="22.86" y1="24.13" x2="24.13" y2="22.86" width="0.1524" layer="16"/>
+<wire x1="24.13" y1="22.86" x2="24.13" y2="15.24" width="0.1524" layer="16"/>
+<wire x1="16.51" y1="32.92" x2="16.51" y2="27.94" width="0.1524" layer="16"/>
+<wire x1="16.51" y1="27.94" x2="20.32" y2="24.13" width="0.1524" layer="16"/>
 </signal>
 </signals>

Commit message: Poligono de Masa a GND
Parts:
- removed X2: (no value), con-wago-500:W237-103
- added LED1: TLLY4400, led:LED3MM
- added R1: (no value), rcl:0204/5
- X1: device con-wago-500:W237-102 -> con-wago-500:W237-4
- moved X1 65.0 mm to (63.5, 35.6), turned to 0 degrees
- moved X6 26.7 mm to (7.62, 35.6)
- moved X7 25.4 mm to (35.6, 35.6)
Connections:
- removed net N$3: SV1.6, X2.3, X6.4, X7.4
- new net GND: LED1.K, SV1.6, X1.4, X6.4, X7.4
- new net N$10: SV6.5, X1.2
- new net N$5: SV6.4, X7.3
- new net N$6: SV6.3, X7.2
- new net N$7: SV6.2, X6.3
- new net N$9: SV6.6, X1.3
- new net TX3: SV6.1, X6.2
- new net VCC: R1.2, SV1.5, X1.1, X6.1, X7.1
- net N$1: now also LED1.A, R1.1; no longer SV1.5, X6.1, X7.1
Routing:
- net VCC: track 0.00 -> 197.7 mm
- net N$1: track 155.3 -> 5.08 mm
- net GND: track 0.00 -> 118.7 mm
- net N$3: track 93.5 -> 0.00 mm
- net TX3: track 0.00 -> 61.2 mm
- net N$7: track 0.00 -> 59.9 mm
- net N$6: track 0.00 -> 41.2 mm
- net N$5: track 0.00 -> 39.5 mm
- net N$9: track 0.00 -> 25.7 mm
- net N$10: track 0.00 -> 24.7 mm
- added copper zone on layer 16, net GND
Other:
- board size 84.8 x 63.5 mm -> 87.3 x 64.8 mm

Commit message: somo titles
Parts:
- renumbered LED1 to INDEX, R1 to 330, X1 to T3, X6 to T1, X7 to T2
Connections:
- net GND: now also SV1.7
Routing:
- net GND: track 118.7 -> 121.3 mm
Other:
- board text added: "5V"
- board text added: "5v"
- board text added: "GND"
- board text added: "RX"
- board text added: "SERIAL 1"
- board text added: "SERIAL 2"
- board text added: "SERIAL 3"
- board text added: "TX"
Changed lines of the file:
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@@
 <drawing>
 <settings>
-<setting alwaysvectorfont="no"/>
+<setting alwaysvectorfont="yes"/>
 <setting verticaltext="up"/>
 </settings>
@@
 <wire x1="79.68" y1="66.03" x2="-7.62" y2="66.03" width="0" layer="20"/>
 <wire x1="-7.62" y1="66.03" x2="-7.62" y2="1.27" width="0" layer="20"/>
+<text x="0" y="44.45" size="1.27" layer="1">SERIAL 1</text>
+<text x="27.94" y="44.45" size="1.27" layer="1">SERIAL 2</text>
+<text x="54.61" y="44.45" size="1.27" layer="1">SERIAL 3</text>
+<text x="-2.54" y="40.64" size="1.27" layer="1">5v</text>
+<text x="13.97" y="40.64" size="1.27" layer="1">GND</text>
+<text x="69.85" y="40.64" size="1.27" layer="1">GND</text>
+<text x="41.91" y="40.64" size="1.27" layer="1">GND</text>
+<text x="25.4" y="40.64" size="1.27" layer="1">5V</text>
+<text x="53.34" y="40.64" size="1.27" layer="1">5V</text>
+<text x="8.89" y="40.64" size="1.27" layer="1">RX</text>
+<text x="3.81" y="40.64" size="1.27" layer="1">TX</text>
+<text x="36.83" y="40.64" size="1.27" layer="1">RX</text>
+<text x="31.75" y="40.64" size="1.27" layer="1">TX</text>
+<text x="64.77" y="40.64" size="1.27" layer="1">RX</text>
+<text x="59.69" y="40.64" size="1.27" layer="1">TX</text>
+<text x="19.05" y="12.7" size="1.27" layer="1" rot="R90">5V</text>
+<text x="24.13" y="12.7" size="1.27" layer="1" rot="R90">GND</text>
 </plain>
 <attributes>
@@
 <attribute name="VALUE" x="57.15" y="55.499" size="1.27" layer="27" ratio="10"/>
 </element>
-<element name="X6" library="con-wago-500" library_urn="urn:adsk.eagle:library:195" package="W237-4" package3d_urn="urn:adsk.eagle:package:10695/1" value="" x="7.62" y="35.56" smashed="yes">
+<element name="T1" library="con-wago-500" library_urn="urn:adsk.eagle:library:195" package="W237-4" package3d_urn="urn:adsk.eagle:package:10695/1" value="" x="7.62" y="35.56" smashed="yes">
 <attribute name="MF" value="" x="7.62" y="35.56" size="1.778" layer="27" display="off"/>
 <attribute name="MPN" value="" x="7.62" y="35.56" size="1.778" layer="27" display="off"/>
@@
 <attribute name="VALUE" x="-0.0324" y="30.5308" size="1.27" layer="27" ratio="10"/>
 </element>
-<element name="X7" library="con-wago-500" library_urn="urn:adsk.eagle:library:195" package="W237-4" package3d_urn="urn:adsk.eagle:package:10695/1" value="" x="35.56" y="35.56" smashed="yes">
+<element name="T2" library="con-wago-500" library_urn="urn:adsk.eagle:library:195" package="W237-4" package3d_urn="urn:adsk.eagle:package:10695/1" value="" x="35.56" y="35.56" smashed="yes">
 <attribute name="MF" value="" x="35.56" y="35.56" size="1.778" layer="27" display="off"/>
 <attribute name="MPN" value="" x="35.56" y="35.56" size="1.778" layer="27" display="off"/>
@@
 <attribute name="VALUE" x="27.9076" y="30.5308" size="1.27" layer="27" ratio="10"/>
 </element>
-<element name="X1" library="con-wago-500" library_urn="urn:adsk.eagle:library:195" package="W237-4" package3d_urn="urn:adsk.eagle:package:10695/1" value="" x="63.5" y="35.56" smashed="yes">
+<element name="T3" library="con-wago-500" library_urn="urn:adsk.eagle:library:195" package="W237-4" package3d_urn="urn:adsk.eagle:package:10695/1" value="" x="63.5" y="35.56" smashed="yes">
 <attribute name="MF" value="" x="63.5" y="35.56" size="1.778" layer="27" display="off"/>
 <attribute name="MPN" value="" x="63.5" y="35.56" size="1.778" layer="27" display="off"/>
@@
 <attribute name="VALUE" x="55.8476" y="30.5308" size="1.27" layer="27" ratio="10"/>
 </element>
-<element name="R1" library="rcl" library_urn="urn:adsk.eagle:library:334" package="0204/5" package3d_urn="urn:adsk.eagle:package:23488/1" value="" x="6.35" y="24.13" smashed="yes" rot="R180">
+<element name="330" library="rcl" library_urn="urn:adsk.eagle:library:334" package="0204/5" package3d_urn="urn:adsk.eagle:package:23488/1" value="" x="6.35" y="24.13" smashed="yes" rot="R180">
 <attribute name="NAME" x="8.3566" y="22.9616" size="0.9906" layer="25" ratio="10" rot="R180"/>
 <attribute name="SPICEPREFIX" value="R" x="6.35" y="24.13" size="1.778" layer="27" rot="R180" display="off"/>
 <attribute name="VALUE" x="8.4836" y="26.4414" size="0.9906" layer="27" ratio="10" rot="R180"/>
 </element>
-<element name="LED1" library="led" library_urn="urn:adsk.eagle:library:259" package="LED3MM" package3d_urn="urn:adsk.eagle:package:15797/1" value="TLLY4400" x="15.24" y="24.13" smashed="yes">
+<element name="INDEX" library="led" library_urn="urn:adsk.eagle:library:259" package="LED3MM" package3d_urn="urn:adsk.eagle:package:15797/1" value="TLLY4400" x="15.24" y="24.13" smashed="yes">
 <attribute name="MF" value="VISHAY SEMICONDUCTOR" x="15.24" y="24.13" size="1.778" layer="27" display="off"/>
 <attribute name="NAME" x="17.145" y="24.511" size="1.27" layer="25" ratio="10"/>
@@
 <signals>
 <signal name="N$5">
-<contactref element="X7" pad="3"/>
+<contactref element="T2" pad="3"/>
 <contactref element="SV6" pad="4"/>
 <wire x1="35.54" y1="34.31" x2="35.56" y2="34.33" width="0.1524" layer="16"/>
@@
 </signal>
 <signal name="N$6">
-<contactref element="X7" pad="2"/>
+<contactref element="T2" pad="2"/>
 <contactref element="SV6" pad="3"/>
 <wire x1="33.06" y1="40.68" x2="33.06" y2="34.29" width="1.27" layer="16"/>
@@
 </signal>
 <signal name="N$7">
-<contactref element="X6" pad="3"/>
+<contactref element="T1" pad="3"/>
 <contactref element="SV6" pad="2"/>
 <wire x1="10.12" y1="34.29" x2="10.12" y2="38.06" width="1.27" layer="16"/>
@@
 </signal>
 <signal name="N$9">
-<contactref element="X1" pad="3"/>
+<contactref element="T3" pad="3"/>
 <contactref element="SV6" pad="6"/>
 <wire x1="62.23" y1="52.07" x2="62.23" y2="58.42" width="1.27" layer="16"/>
@@
 </signal>
 <signal name="N$10">
-<contactref element="X1" pad="2"/>
+<contactref element="T3" pad="2"/>
 <contactref element="SV6" pad="5"/>
 <wire x1="59.69" y1="49.53" x2="60.96" y2="48.26" width="1.27" layer="16"/>
@@
 </signal>
 <signal name="TX3">
-<contactref element="X6" pad="2"/>
+<contactref element="T1" pad="2"/>
 <contactref element="SV6" pad="1"/>
 <wire x1="48.26" y1="50.8" x2="33.02" y2="50.8" width="1.27" layer="16"/>
@@
 </signal>
 <signal name="GND">
-<contactref element="X6" pad="4"/>
-<contactref element="X7" pad="4"/>
+<contactref element="T1" pad="4"/>
+<contactref element="T2" pad="4"/>
 <contactref element="SV1" pad="6"/>
-<contactref element="X1" pad="4"/>
+<contactref element="T3" pad="4"/>
 <wire x1="15.12" y1="34.29" x2="16.39" y2="35.56" width="0.1524" layer="16"/>
 <wire x1="16.39" y1="35.56" x2="16.51" y2="35.56" width="0.1524" layer="16"/>
@@
 <wire x1="40.64" y1="29.21" x2="38.1" y2="26.67" width="1.27" layer="16"/>
 <wire x1="38.1" y1="26.67" x2="30.48" y2="26.67" width="1.27" layer="16"/>
-<wire x1="29.845" y1="26.035" x2="27.94" y2="24.13" width="1.27" layer="16"/>
+<wire x1="30.48" y1="26.67" x2="27.94" y2="24.13" width="1.27" layer="16"/>
 <wire x1="43.06" y1="34.29" x2="44.45" y2="34.29" width="1.27" layer="16"/>
 <wire x1="48.26" y1="30.48" x2="48.26" y2="29.21" width="1.27" layer="16"/>
@@
 <vertex x="78.74" y="63.5"/>
 </polygon>
-<contactref element="LED1" pad="K"/>
+<contactref element="INDEX" pad="K"/>
 <wire x1="16.51" y1="24.13" x2="19.05" y2="24.13" width="1.27" layer="16"/>
 <wire x1="19.05" y1="24.13" x2="21.59" y2="21.59" width="1.27" layer="16"/>
 <wire x1="21.59" y1="21.59" x2="21.59" y2="10.16" width="1.27" layer="16"/>
-<wire x1="30.48" y1="26.67" x2="29.845" y2="26.035" width="1.27" layer="16"/>
 <wire x1="30.48" y1="36.83" x2="30.48" y2="26.67" width="1.27" layer="16"/>
 <polygon width="1.016" layer="16" isolate="0.8128">
@@
 <vertex x="78.74" y="64.77"/>
 </polygon>
+<contactref element="SV1" pad="7"/>
+<wire x1="24.13" y1="10.16" x2="21.59" y2="10.16" width="1.016" layer="16"/>
 </signal>
 <signal name="VCC">
-<contactref element="X6" pad="1"/>
-<contactref element="X7" pad="1"/>
+<contactref element="T1" pad="1"/>
+<contactref element="T2" pad="1"/>
 <contactref element="SV1" pad="5"/>
-<contactref element="X1" pad="1"/>
+<contactref element="T3" pad="1"/>
 <wire x1="22.86" y1="27.94" x2="1.27" y2="27.94" width="1.27" layer="16"/>
 <wire x1="1.27" y1="27.94" x2="0" y2="29.21" width="1.27" layer="16"/>
@@
 <wire x1="27.94" y1="34.17" x2="27.94" y2="33.02" width="1.27" layer="16"/>
 <wire x1="27.94" y1="33.02" x2="22.86" y2="27.94" width="1.27" layer="16"/>
-<contactref element="R1" pad="2"/>
+<contactref element="330" pad="2"/>
 <wire x1="19.05" y1="10.16" x2="19.05" y2="13.97" width="1.27" layer="16"/>
 <wire x1="15.24" y1="17.78" x2="1.27" y2="17.78" width="1.27" layer="16"/>
@@
 </signal>
 <signal name="N$1">
-<contactref element="LED1" pad="A"/>
-<contactref element="R1" pad="1"/>
+<contactref element="INDEX" pad="A"/>
+<contactref element="330" pad="1"/>
 <wire x1="8.89" y1="24.13" x2="13.97" y2="24.13" width="1.27" layer="16"/>
 </signal>
